File: Electronics/breakout.sch (EAGLE design)
At the start: 7 parts, among them J1 FLATPACK2_CON, J4 FLATPACK2_DC_LUG, J5 FLATPACK2_DC_LUG, J6 FLATPACK2_DC_LUG, J7 FLATPACK2_DC_LUG

Commit message: Lots of changes; final board revision
Parts:
- J3: device SparkFun-Connectors:CONN_02POGO_PIN_HOLES_ONLY -> SparkFun-Connectors:CONN_021X02_NO_SILK
Changed lines of the file:
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@@
 <parts>
 <part name="J1" library="flatpack2-edge-connector" deviceset="FLATPACK2_CON" device=""/>
-<part name="J3" library="SparkFun-Connectors" deviceset="CONN_02" device="POGO_PIN_HOLES_ONLY"/>
+<part name="J3" library="SparkFun-Connectors" deviceset="CONN_02" device="1X02_NO_SILK"/>
 <part name="J2" library="connectors" deviceset="WEIDMULLER_PM_508" device=""/>
 <part name="J4" library="connectors" deviceset="FLATPACK2_DC_LUG" device=""/>

Commit message: Final revision of Flatpack breakout PCB
Connections:
- removed net N$4 (its old number): J1.AC_ACTIVE, J2.1
- new net N$3: J1.AC_LIVE, J2.1
- new net N$6: J1.AC_EARTH, J2.3
Changed lines of the file:
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@@
 <part name="J1" library="flatpack2-edge-connector" deviceset="FLATPACK2_CON" device=""/>
 <part name="J3" library="SparkFun-Connectors" deviceset="CONN_02" device="1X02_NO_SILK"/>
-<part name="J2" library="connectors" deviceset="WEIDMULLER_PM_508" device=""/>
 <part name="J4" library="connectors" deviceset="FLATPACK2_DC_LUG" device=""/>
 <part name="J5" library="connectors" deviceset="FLATPACK2_DC_LUG" device=""/>
 <part name="J6" library="connectors" deviceset="FLATPACK2_DC_LUG" device=""/>
 <part name="J7" library="connectors" deviceset="FLATPACK2_DC_LUG" device=""/>
+<part name="J2" library="connectors" deviceset="WEIDMULLER_PM_508" device=""/>
 </parts>
 <sheets>
@@
 <instance part="J1" gate="G$1" x="22.86" y="2.54"/>
 <instance part="J3" gate="G$1" x="35.56" y="17.78" rot="R180"/>
-<instance part="J2" gate="G$1" x="35.56" y="7.62" rot="R180"/>
 <instance part="J4" gate="G$1" x="40.64" y="17.78" rot="R270"/>
 <instance part="J5" gate="G$1" x="43.18" y="17.78" rot="R270"/>
 <instance part="J6" gate="G$1" x="45.72" y="17.78" rot="R270"/>
 <instance part="J7" gate="G$1" x="48.26" y="17.78" rot="R270"/>
+<instance part="J2" gate="G$1" x="35.56" y="2.54" rot="R180"/>
 </instances>
 <busses>
@@
 <wire x1="25.4" y1="12.7" x2="22.86" y2="12.7" width="0.1524" layer="91"/>
 <pinref part="J3" gate="G$1" pin="2"/>
-</segment>
-</net>
-<net name="N$3" class="0">
-<segment>
-<pinref part="J1" gate="G$1" pin="AC_NEUTRAL"/>
-<wire x1="22.86" y1="2.54" x2="25.4" y2="2.54" width="0.1524" layer="91"/>
-<wire x1="25.4" y1="2.54" x2="25.4" y2="5.08" width="0.1524" layer="91"/>
-<pinref part="J2" gate="G$1" pin="2"/>
-<wire x1="25.4" y1="5.08" x2="27.94" y2="5.08" width="0.1524" layer="91"/>
-</segment>
-</net>
-<net name="N$4" class="0">
-<segment>
-<pinref part="J2" gate="G$1" pin="1"/>
-<pinref part="J1" gate="G$1" pin="AC_ACTIVE"/>
-<wire x1="27.94" y1="7.62" x2="22.86" y2="7.62" width="0.1524" layer="91"/>
 </segment>
 </net>
@@
 </segment>
 </net>
+<net name="N$3" class="0">
+<segment>
+<pinref part="J1" gate="G$1" pin="AC_LIVE"/>
+<wire x1="22.86" y1="7.62" x2="25.4" y2="7.62" width="0.1524" layer="91"/>
+<wire x1="25.4" y1="7.62" x2="25.4" y2="5.08" width="0.1524" layer="91"/>
+<pinref part="J2" gate="G$1" pin="1"/>
+<wire x1="25.4" y1="5.08" x2="27.94" y2="5.08" width="0.1524" layer="91"/>
+</segment>
+</net>
+<net name="N$4" class="0">
+<segment>
+<pinref part="J2" gate="G$1" pin="2"/>
+<pinref part="J1" gate="G$1" pin="AC_NEUTRAL"/>
+<wire x1="27.94" y1="2.54" x2="22.86" y2="2.54" width="0.1524" layer="91"/>
+</segment>
+</net>
+<net name="N$6" class="0">
+<segment>
+<pinref part="J1" gate="G$1" pin="AC_EARTH"/>
+<wire x1="22.86" y1="-2.54" x2="25.4" y2="-2.54" width="0.1524" layer="91"/>
+<wire x1="25.4" y1="-2.54" x2="25.4" y2="0" width="0.1524" layer="91"/>
+<pinref part="J2" gate="G$1" pin="3"/>
+<wire x1="25.4" y1="0" x2="27.94" y2="0" width="0.1524" layer="91"/>
+</segment>
+</net>
